File: PCB/ADX-ddsPIO.kicad_sch (KiCad schematic)
At the start: 79 parts, among them J1 Conn_Coaxial, J2 +12V, J3 SPKR, J4 MIC, Q1 BS170, Q2 BS170, Q3 BS170, Q4 BS170, Q5 BS170, U1 L7805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

Commit message: doc
Connections:
- net RXOSC: now also U3.2 (GP1)
- net at JP1.2 (C): now also U3.16 (GP12); no longer U3.19 (GP14)
- net at R19.2, SYNC.3 (B), SYNC.4 (B): now also U3.17 (GP13)
- net at R5.1: now also U3.9 (GP6); no longer U3.10 (GP7)
- net at R8.2, UP.3 (B), UP.4 (B): now also U3.14 (GP10); no longer U3.15 (GP11)
- net at R9.2, TX.3 (B), TX.4 (B): now also U3.11 (GP8); no longer U3.14 (GP10)
- net at C2.1: now also U3.1 (GP0); no longer U3.9 (GP6)
- net at DOWN.3 (B), DOWN.4 (B), R7.2: now also U3.15 (GP11); no longer U3.16 (GP12)
- net at R6.1: now also U3.10 (GP7); no longer U3.11 (GP8)
Changed lines of the file:
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@@
   (junction (at 194.31 101.6) (diameter 0) (color 0 0 0 0)
   )
+  (junction (at 83.82 154.94) (diameter 0) (color 0 0 0 0)
+  )
   (junction (at 137.16 142.24) (diameter 0) (color 0 0 0 0)
   )
@@
   (junction (at 97.79 127) (diameter 0) (color 0 0 0 0)
   )
+  (junction (at 52.07 119.38) (diameter 0) (color 0 0 0 0)
+  )
   (junction (at 137.16 144.78) (diameter 0) (color 0 0 0 0)
   )
@@
     (stroke (width 0) (type default))
   )
-  (wire (pts (xy 49.53 154.94) (xy 49.53 175.26))
+  (wire (pts (xy 49.53 152.4) (xy 49.53 175.26))
     (stroke (width 0) (type default))
   )
@@
     (stroke (width 0) (type default))
   )
+  (wire (pts (xy 49.53 96.52) (xy 72.39 96.52))
+    (stroke (width 0) (type default))
+  )
   (wire (pts (xy 199.39 48.26) (xy 201.93 48.26))
     (stroke (width 0) (type default))
@@
     (stroke (width 0) (type default))
   )
-  (wire (pts (xy 52.07 149.86) (xy 46.99 149.86))
+  (wire (pts (xy 83.82 154.94) (xy 80.01 154.94))
     (stroke (width 0) (type default))
   )
@@
     (stroke (width 0) (type default))
   )
-  (wire (pts (xy 48.26 152.4) (xy 48.26 176.53))
+  (wire (pts (xy 48.26 149.86) (xy 48.26 176.53))
     (stroke (width 0) (type default))
   )
@@
     (stroke (width 0) (type default))
   )
+  (wire (pts (xy 52.07 118.11) (xy 52.07 119.38))
+    (stroke (width 0) (type default))
+  )
   (wire (pts (xy 77.47 147.32) (xy 78.74 147.32))
     (stroke (width 0) (type default))
@@
     (stroke (width 0) (type default))
   )
+  (wire (pts (xy 80.01 181.61) (xy 45.72 181.61))
+    (stroke (width 0) (type default))
+  )
   (wire (pts (xy 77.47 134.62) (xy 78.74 134.62))
     (stroke (width 0) (type default))
@@
     (stroke (width 0) (type default))
   )
+  (wire (pts (xy 52.07 139.7) (xy 40.64 139.7))
+    (stroke (width 0) (type default))
+  )
   (wire (pts (xy 111.76 96.52) (xy 111.76 129.54))
     (stroke (width 0) (type default))
@@
     (stroke (width 0) (type default))
   )
+  (wire (pts (xy 52.07 149.86) (xy 48.26 149.86))
+    (stroke (width 0) (type default))
+  )
   (wire (pts (xy 153.67 101.6) (xy 161.29 101.6))
     (stroke (width 0) (type default))
@@
     (stroke (width 0) (type default))
   )
+  (wire (pts (xy 80.01 154.94) (xy 80.01 181.61))
+    (stroke (width 0) (type default))
+  )
   (wire (pts (xy 111.76 142.24) (xy 111.76 144.78))
     (stroke (width 0) (type default))
@@
     (stroke (width 0) (type default))
   )
-  (wire (pts (xy 44.45 162.56) (xy 44.45 175.26))
+  (wire (pts (xy 52.07 142.24) (xy 46.99 142.24))
+    (stroke (width 0) (type default))
+  )
+  (wire (pts (xy 44.45 154.94) (xy 44.45 175.26))
     (stroke (width 0) (type default))
   )
@@
     (stroke (width 0) (type default))
   )
-  (wire (pts (xy 34.29 139.7) (xy 52.07 139.7))
+  (wire (pts (xy 52.07 119.38) (xy 30.48 119.38))
     (stroke (width 0) (type default))
   )
@@
     (stroke (width 0) (type default))
   )
+  (wire (pts (xy 45.72 181.61) (xy 45.72 157.48))
+    (stroke (width 0) (type default))
+  )
   (wire (pts (xy 78.74 121.92) (xy 78.74 134.62))
     (stroke (width 0) (type default))
@@
     (stroke (width 0) (type default))
   )
+  (wire (pts (xy 49.53 116.84) (xy 49.53 96.52))
+    (stroke (width 0) (type default))
+  )
   (wire (pts (xy 213.36 43.18) (xy 226.06 43.18))
     (stroke (width 0) (type default))
@@
     (stroke (width 0) (type default))
   )
-  (wire (pts (xy 39.37 137.16) (xy 52.07 137.16))
+  (wire (pts (xy 34.29 137.16) (xy 52.07 137.16))
     (stroke (width 0) (type default))
   )
@@
     (stroke (width 0) (type default))
   )
+  (wire (pts (xy 40.64 139.7) (xy 40.64 148.59))
+    (stroke (width 0) (type default))
+  )
   (wire (pts (xy 78.74 147.32) (xy 78.74 160.02))
     (stroke (width 0) (type default))
@@
     (stroke (width 0) (type default))
   )
+  (wire (pts (xy 52.07 154.94) (xy 44.45 154.94))
+    (stroke (width 0) (type default))
+  )
   (wire (pts (xy 46.99 24.13) (xy 46.99 29.21))
     (stroke (width 0) (type default))
   )
+  (wire (pts (xy 52.07 152.4) (xy 49.53 152.4))
+    (stroke (width 0) (type default))
+  )
   (wire (pts (xy 162.56 76.2) (xy 162.56 83.82))
     (stroke (width 0) (type default))
@@
     (stroke (width 0) (type default))
   )
-  (wire (pts (xy 72.39 96.52) (xy 39.37 96.52))
-    (stroke (width 0) (type default))
-  )
   (wire (pts (xy 162.56 76.2) (xy 157.48 76.2))
     (stroke (width 0) (type default))
@@
     (stroke (width 0) (type default))
   )
-  (wire (pts (xy 39.37 96.52) (xy 39.37 137.16))
+  (wire (pts (xy 83.82 154.94) (xy 83.82 156.21))
     (stroke (width 0) (type default))
   )
@@
     (stroke (width 0) (type default))
   )
-  (wire (pts (xy 83.82 152.4) (xy 83.82 156.21))
+  (wire (pts (xy 83.82 152.4) (xy 83.82 154.94))
     (stroke (width 0) (type default))
   )
@@
     (stroke (width 0) (type default))
   )
-  (wire (pts (xy 40.64 142.24) (xy 52.07 142.24))
-    (stroke (width 0) (type default))
-  )
   (wire (pts (xy 205.74 55.88) (xy 205.74 63.5))
     (stroke (width 0) (type default))
@@
     (stroke (width 0) (type default))
   )
-  (wire (pts (xy 40.64 148.59) (xy 40.64 142.24))
-    (stroke (width 0) (type default))
-  )
   (wire (pts (xy 193.04 64.77) (xy 201.93 64.77))
     (stroke (width 0) (type default))
@@
     (stroke (width 0) (type default))
   )
+  (wire (pts (xy 45.72 157.48) (xy 52.07 157.48))
+    (stroke (width 0) (type default))
+  )
   (wire (pts (xy 64.77 170.18) (xy 64.77 171.45))
     (stroke (width 0) (type default))
@@
     (stroke (width 0) (type default))
   )
-  (wire (pts (xy 44.45 162.56) (xy 52.07 162.56))
-    (stroke (width 0) (type default))
-  )
   (wire (pts (xy 162.56 68.58) (xy 157.48 68.58))
     (stroke (width 0) (type default))
@@
     (stroke (width 0) (type default))
   )
-  (wire (pts (xy 46.99 149.86) (xy 46.99 177.8))
+  (wire (pts (xy 46.99 142.24) (xy 46.99 177.8))
     (stroke (width 0) (type default))
   )
@@
     (stroke (width 0) (type default))
   )
-  (wire (pts (xy 34.29 148.59) (xy 34.29 139.7))
+  (wire (pts (xy 34.29 137.16) (xy 34.29 148.59))
     (stroke (width 0) (type default))
   )
@@
     (stroke (width 0) (type default))
   )
-  (wire (pts (xy 52.07 152.4) (xy 48.26 152.4))
+  (wire (pts (xy 52.07 116.84) (xy 49.53 116.84))
     (stroke (width 0) (type default))
   )
@@
   )
   (wire (pts (xy 124.46 101.6) (xy 124.46 121.92))
-    (stroke (width 0) (type default))
-  )
-  (wire (pts (xy 52.07 154.94) (xy 49.53 154.94))
     (stroke (width 0) (type default))
   )
@@
     )
   )
+  (global_label "RXOSC" (shape input) (at 30.48 119.38 180) (fields_autoplaced)
+    (effects (font (size 1.27 1.27)) (justify right))
+    (property "Intersheetrefs" "${INTERSHEET_REFS}" (at 21.2847 119.38 0)
+      (effects (font (size 1.27 1.27)) (justify right) hide)
+    )
+  )

Commit message: doc
Changed lines of the file:
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@@
     (stroke (width 0) (type default))
   )
-  (wire (pts (xy 80.01 181.61) (xy 45.72 181.61))
+  (wire (pts (xy 80.01 179.07) (xy 45.72 179.07))
     (stroke (width 0) (type default))
   )
@@
     (stroke (width 0) (type default))
   )
-  (wire (pts (xy 124.46 162.56) (xy 124.46 166.37))
+  (wire (pts (xy 124.46 162.56) (xy 124.46 175.26))
     (stroke (width 0) (type default))
   )
@@
     (stroke (width 0) (type default))
   )
-  (wire (pts (xy 80.01 154.94) (xy 80.01 181.61))
+  (wire (pts (xy 80.01 154.94) (xy 80.01 179.07))
     (stroke (width 0) (type default))
   )
@@
     (stroke (width 0) (type default))
   )
-  (wire (pts (xy 45.72 181.61) (xy 45.72 157.48))
+  (wire (pts (xy 45.72 179.07) (xy 45.72 157.48))
     (stroke (width 0) (type default))
   )
@@
     (effects (font (size 1.27 1.27)) (justify left bottom))
   )
-  (text "WSPR" (at 39.37 168.91 0)
+  (text "WSPR" (at 38.1 168.91 0)
     (effects (font (size 1.27 1.27)) (justify left bottom))
   )
@@
     )
   )
-  (symbol (lib_id "power:GND") (at 124.46 166.37 0) (unit 1)
+  (symbol (lib_id "power:GND") (at 124.46 175.26 0) (unit 1)
     (in_bom yes) (on_board yes) (dnp no) (fields_autoplaced)
-    (property "Reference" "#PWR01" (at 124.46 172.72 0)
-      (effects (font (size 1.27 1.27)) hide)
-    )
-    (property "Value" "GND" (at 124.46 171.45 0)
-      (effects (font (size 1.27 1.27)) hide)
-    )
-    (property "Footprint" "" (at 124.46 166.37 0)
-      (effects (font (size 1.27 1.27)) hide)
-    )
-    (property "Datasheet" "" (at 124.46 166.37 0)
-      (effects (font (size 1.27 1.27)) hide)
-    )
+    (property "Reference" "#PWR01" (at 124.46 181.61 0)
+      (effects (font (size 1.27 1.27)) hide)
+    )
+    (property "Value" "GND" (at 124.46 180.34 0)
+      (effects (font (size 1.27 1.27)) hide)
+    )
+    (property "Footprint" "" (at 124.46 175.26 0)
+      (effects (font (size 1.27 1.27)) hide)
+    )
+    (property "Datasheet" "" (at 124.46 175.26 0)
+      (effects (font (size 1.27 1.27)) hide)
+    )

Commit message: RFOUT
Parts:
- added TP6: RFOUT, symbol Connector:TestPoint
- added TP7: RF Driver, symbol Connector:TestPoint
Connections:
- net GND: now also R10.1, R15.1, R18.1, R19.1, R7.1, R8.1, R9.1
- net RXOSC: now also U3.26 (GP20); no longer U3.2 (GP1)
- net at C1.2, D1.1 (K), Q1.2 (G)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: now also TP7.1
- net at C2.1: now also U3.24 (GP18), TP6.1; no longer U3.1 (GP0)
- removed net +3.3V: R10.1, R15.1, R18.1, R19.1, R7.1, R8.1, R9.1, U3.36 (3V3(OUT))
Other:
- moved on the sheet: C2, D4, D5, D6, D7, D8, DOWN, JP1, R18, R19, R2, R3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

Commit message: testADX
Parts:
- removed C10, C7: 100n, symbol Device:C
- removed C11: 470n, symbol Device:C
- removed C8, C9: 10n, symbol Device:C
- removed J3: SPKR, symbol Connector_Audio:AudioJack2
- removed J4: MIC, symbol Connector_Audio:AudioJack2
- removed Q4: BS170, Package_TO_SOT_THT:TO-92_Inline, symbol Transistor_FET:BS170
- removed R10: 1M, symbol Device:R
- removed R11, R12, R13: 10K, symbol Device:R
- removed R14: 100K, symbol Device:R
- removed R15: 1K, symbol Device:R
- removed TP6: RFOUT, symbol Connector:TestPoint
- added Q6, Q7: BS170, Package_TO_SOT_THT:TO-92_Inline, symbol Transistor_FET:BS170
- added TP8: RXOSC, symbol Connector:TestPoint
- added TP9: TXOSC, symbol Connector:TestPoint
Connections:
- net RXOSC: now also Q6.3 (S), TP8.1
- net RXSW: now also Q6.2 (G)
- net at U3.24 (GP18): now also Q6.1 (D), Q7.1 (D); no longer C2.1
- net TXOSC: now reaches C2.2, U2.11 (I0b), U2.13 (I1b), U2.15 (I2b), U2.17 (I3b), U2.2 (I0a), U2.4 (I1a), U2.6 (I2a), U2.8 (I3a)
- net TXOSC: now also TP9.1
- net at R2.1, U3.5 (GP3): now also Q7.2 (G)
- net FSK: no longer names the net of U3.32 (GP27)
- new net: C2.1, Q7.3 (S)
Other:
- moved on the sheet: C2

Commit message: PCB
Parts:
- added C10, C11: 10n, symbol Device:C
- added C7, C8: 100n, symbol Device:C
- added C9: 470n, symbol Device:C
- added J3: SPKR, symbol Connector_Audio:AudioJack2
- added J4: MIC, symbol Connector_Audio:AudioJack2
- added J5: Serial Monitor, symbol Connector_Generic:Conn_01x02
- added JP2: analog/digital, symbol Jumper:Jumper_2_Bridged
- added JP3: Jumper_3_Bridged12, symbol Jumper:Jumper_3_Bridged12
- added Q4: BS170, Package_TO_SOT_THT:TO-92_Inline, symbol Transistor_FET:BS170
- added R10: 1M, symbol Device:R
- added R11, R12, R13: 10K, symbol Device:R
- added R14: 100K, symbol Device:R
- added R15: 1K, symbol Device:R
- added TP10: RXA, symbol Connector:TestPoint
- added TP6: FSK, symbol Connector:TestPoint
Connections:
- net GND: now also C10.2, C11.2, C8.2, Q4.3 (S), R10.1, R11.2, R14.2, R15.1
- net RXA: now also JP3.2 (C), TP10.1
- net at U3.1 (GP0): now also J5.2 (Pin_2)
- net at U3.2 (GP1): now also J5.1 (Pin_1)
- net at U3.31 (GP26): now also JP3.1 (A)
- net at U3.32 (GP27): now also JP2.1 (A)
- new net: C11.1, Q4.2 (G), R13.2, R14.1
- new net: C9.2, JP3.3 (B)
- new net: C7.1, J3.S, J3.T
- new net: C7.2, R10.2, R11.1, R12.1
- new net: C8.1, C9.1, J4.S, J4.T
- new net: C10.1, R12.2, R13.1
- new net FSK: JP2.2 (B), Q4.1 (D), R15.2, TP6.1

Commit message: ADX-ddsPIO
Connections:
- net RXOSC: no longer U3.26 (GP20)
- net RFOUT: now reaches Q6.1 (D), Q7.1 (D), U3.24 (GP18)
Changed lines of the file:
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@@
   (junction (at 41.91 38.1) (diameter 0) (color 0 0 0 0)
   )
+  (junction (at 83.82 157.48) (diameter 0) (color 0 0 0 0)
+  )
   (junction (at 166.37 83.82) (diameter 0) (color 0 0 0 0)
   )
@@
     (stroke (width 0) (type default))
   )
-  (wire (pts (xy 76.2 152.4) (xy 87.63 152.4))
-    (stroke (width 0) (type default))
-  )
   (wire (pts (xy 111.76 85.09) (xy 120.65 85.09))
     (stroke (width 0) (type default))
@@
   )
   (wire (pts (xy 137.16 144.78) (xy 137.16 147.32))
+    (stroke (width 0) (type default))
+  )
+  (wire (pts (xy 83.82 157.48) (xy 87.63 157.48))
     (stroke (width 0) (type default))
   )
@@
     )
   )
-  (global_label "RXOSC" (shape input) (at 87.63 152.4 0) (fields_autoplaced)
+  (global_label "RFOUT" (shape input) (at 87.63 157.48 0) (fields_autoplaced)
     (effects (font (size 1.27 1.27)) (justify left))
-    (property "Intersheetrefs" "${INTERSHEET_REFS}" (at 96.8253 152.4 0)
+    (property "Intersheetrefs" "${INTERSHEET_REFS}" (at 96.523 157.48 0)
       (effects (font (size 1.27 1.27)) (justify left) hide)
     )

Commit message: ADX-ddsPIO_SW_n_LED
Parts:
- removed C10, C11: 10n, symbol Device:C
- removed C7, C8: 100n, symbol Device:C
- removed C9: 470n, symbol Device:C
- removed J3: SPKR, symbol Connector_Audio:AudioJack2
- removed J4: MIC, symbol Connector_Audio:AudioJack2
- removed J5: Serial Monitor, symbol Connector_Generic:Conn_01x02
- removed JP2: analog/digital, symbol Jumper:Jumper_2_Bridged
- removed JP3: Jumper_3_Bridged12, symbol Jumper:Jumper_3_Bridged12
- removed Q4: BS170, Package_TO_SOT_THT:TO-92_Inline, symbol Transistor_FET:BS170
- removed R10: 1M, symbol Device:R
- removed R11, R12, R13: 10K, symbol Device:R
- removed R14: 100K, symbol Device:R
- removed R15: 1K, symbol Device:R
- removed TP10: RXA, symbol Connector:TestPoint
- removed TP6: FSK, symbol Connector:TestPoint
Connections:
- net RXA: now also U3.31 (GP26)

Commit message: ADX-ddsPIO_rp2040Z
Parts:
- removed Q6, Q7: BS170, Package_TO_SOT_THT:TO-92_Inline, symbol Transistor_FET:BS170
- removed TP2: CAL, symbol Connector:TestPoint
- removed TP9: TXOSC, symbol Connector:TestPoint
- added C7: 100n, symbol Device:C
- added R10: 1K, symbol Device:R
- C2: value 10n -> 100n
Connections:
- net RXOSC is gone; now on net RFOUT: C20.1, TP8.1
- net +5V: now also C7.1
- net GND: now also C7.2, R10.1; no longer U2.1 (OEa), U2.19 (OEb)
- net RFOUT: now also C2.1
- net TXA: now reaches U3.12 (GP9)
- net TXA: now also U2.1 (OEa), U2.19 (OEb), R10.2
- net TXOSC: no longer names the net of C2.2, U2.11 (I0b), U2.13 (I1b), U2.15 (I2b), U2.17 (I3b), U2.2 (I0a), U2.4 (I1a), U2.6 (I2a), U2.8 (I3a)
Other:
- moved on the sheet: C2
