File: PCB/ADX-ddsPIO.kicad_sch (KiCad schematic)
At the start: 68 parts, among them J1 Conn_Coaxial, J2 +12V, Q1 BS170, Q2 BS170, Q3 BS170, Q5 BS170, U1 L7805, U2 74LS244, U4 CD2003GB_GP

Commit message: ADX-ddsPIO-V1.0
Parts:
- added C8: 470n, symbol Device:C
- added R11, R12: 10K, symbol Device:R
- added TP2: +3.3V, symbol Connector:TestPoint
Connections:
- net GND: now also R10.2, R11.2, R12.1, TP2.1; no longer R10.1, R18.1, R19.1, R7.1, R8.1, R9.1
- net RFOUT: no longer C2.1, C20.1, TP8.1, U3.24 (GP18)
- net RXA: now also C8.1, R11.1, R12.2; no longer U4.4 (AM_MIX)
- net TXA: now also R10.1; no longer R10.2
- net at JP1.2 (C): now also U3.17 (GP13); no longer U3.16 (GP12)
- net at R19.2, SYNC.3 (B), SYNC.4 (B): now also U3.16 (GP12); no longer U3.17 (GP13)
- net at U3.19 (GP14): now also C2.1
- net at U3.20 (GP15): no longer TP3.1
- new net: C8.2, U4.4 (AM_MIX)
- new net: C20.1, TP8.1
- new net +3.3V: R18.1, R19.1, R7.1, R8.1, R9.1
Other:
- moved on the sheet: C2, C20, DOWN, JP1, R10, R18, R19, R7, R8, R9, SYNC, TP3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

Commit message: ADX-ddsPIO-V1.0
Parts:
- TP3: value ATU -> DCO
Connections:
- net RFOUT: now also C2.1, TP3.1, U3.19 (GP14)
Other:
- moved on the sheet: TP3
Changed lines of the file:
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@@
   (title_block
     (date "Dec,27 2025")
-    (rev "0.1")
+    (rev "1.0")
   )
   (junction (at 27.94 55.88) (diameter 0) (color 0 0 0 0)
@@
   (junction (at 194.31 101.6) (diameter 0) (color 0 0 0 0)
   )
+  (junction (at 81.28 177.8) (diameter 0) (color 0 0 0 0)
+  )
   (junction (at 137.16 142.24) (diameter 0) (color 0 0 0 0)
   )
@@
   (junction (at 21.59 69.85) (diameter 0) (color 0 0 0 0)
   )
+  (junction (at 88.9 166.37) (diameter 0) (color 0 0 0 0)
+  )
   (junction (at 111.76 25.4) (diameter 0) (color 0 0 0 0)
   )
@@
     (stroke (width 0) (type default))
   )
+  (wire (pts (xy 88.9 166.37) (xy 91.44 166.37))
+    (stroke (width 0) (type default))
+  )
   (wire (pts (xy 111.76 139.7) (xy 111.76 142.24))
     (stroke (width 0) (type default))
@@
     (stroke (width 0) (type default))
   )
-  (wire (pts (xy 45.72 177.8) (xy 88.9 177.8))
+  (wire (pts (xy 45.72 177.8) (xy 81.28 177.8))
     (stroke (width 0) (type default))
   )
@@
     (stroke (width 0) (type default))
   )
+  (wire (pts (xy 81.28 177.8) (xy 88.9 177.8))
+    (stroke (width 0) (type default))
+  )
   (wire (pts (xy 63.5 171.45) (xy 49.53 171.45))
     (stroke (width 0) (type default))
@@
     (stroke (width 0) (type default))
   )
-  (wire (pts (xy 88.9 147.32) (xy 88.9 177.8))
+  (wire (pts (xy 88.9 147.32) (xy 88.9 166.37))
     (stroke (width 0) (type default))
   )
@@
     (stroke (width 0) (type default))
   )
+  (wire (pts (xy 88.9 166.37) (xy 88.9 177.8))
+    (stroke (width 0) (type default))
+  )
   (wire (pts (xy 100.33 101.6) (xy 124.46 101.6))
     (stroke (width 0) (type default))
@@
     )
   )
-  (global_label "RFOUT" (shape input) (at 118.11 195.58 0) (fields_autoplaced)
+  (global_label "RFOUT" (shape input) (at 91.44 166.37 0) (fields_autoplaced)
     (effects (font (size 1.27 1.27)) (justify left))
-    (property "Intersheetrefs" "${INTERSHEET_REFS}" (at 127.003 195.58 0)
+    (property "Intersheetrefs" "${INTERSHEET_REFS}" (at 100.333 166.37 0)
       (effects (font (size 1.27 1.27)) (justify left) hide)
     )
@@
     )
   )
-  (symbol (lib_id "Connector:TestPoint") (at 74.93 193.04 180) (unit 1)
+  (symbol (lib_id "Connector:TestPoint") (at 81.28 177.8 0) (unit 1)
     (in_bom yes) (on_board yes) (dnp no)
-    (property "Reference" "TP3" (at 80.01 194.31 0)
+    (property "Reference" "TP3" (at 83.82 171.45 0)
       (effects (font (size 1.27 1.27)) (justify left))
     )
-    (property "Value" "ATU" (at 80.01 191.77 0)
+    (property "Value" "DCO" (at 83.82 173.99 0)
       (effects (font (size 1.27 1.27)) (justify left))
     )
-    (property "Footprint" "" (at 69.85 193.04 0)
+    (property "Footprint" "" (at 86.36 177.8 0)
       (effects (font (size 1.27 1.27)) hide)
     )
-    (property "Datasheet" "~" (at 69.85 193.04 0)
+    (property "Datasheet" "~" (at 86.36 177.8 0)
       (effects (font (size 1.27 1.27)) hide)
     )

Commit message: ADX-ddsPIO_V1.2
Parts:
- removed R18: 10K, symbol Device:R
- added TP6: RXIF, symbol Connector:TestPoint
- JP1: value Beacon -> RX Clock
- TP8: value RXOSC -> RXLO
Connections:
- net GND: no longer JP1.1 (A)
- net RFOUT: now also JP1.1 (A)
- net at JP1.2 (C): now also C20.1, TP8.1; no longer U3.17 (GP13)
- net at JP1.3 (B): now also U3.17 (GP13)
- net RXIF: now reaches U3.20 (GP15)
- net RXIF: now also TP6.1
Other:
- moved on the sheet: TP3
