File: PCB/ADX-ddsPIO.kicad_sch (KiCad schematic)
At the start: 72 parts, among them J1 Conn_Coaxial, J2 +12V, Q1 BS170, Q2 BS170, Q3 BS170, Q5 BS170, U1 L7805, U2 74LS244, U4 CD2003GB_GP

Commit message: fix_DualClk
Parts:
- removed JP1: RX Clock, symbol Jumper:Jumper_3_Bridged12
Connections:
- net at C20.1, TP8.1: now also U3.17 (GP13)
Changed lines of the file:
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@@
   (junction (at 49.53 134.62) (diameter 0) (color 0 0 0 0)
   )
-  (junction (at 96.52 147.32) (diameter 0) (color 0 0 0 0)
-  )
   (junction (at 250.19 43.18) (diameter 0) (color 0 0 0 0)
   )
@@
   (junction (at 137.16 139.7) (diameter 0) (color 0 0 0 0)
   )
-  (junction (at 83.82 100.33) (diameter 0) (color 0 0 0 0)
-  )
   (junction (at 111.76 147.32) (diameter 0) (color 0 0 0 0)
   )
@@
     (stroke (width 0) (type default))
   )
+  (wire (pts (xy 90.17 100.33) (xy 43.18 100.33))
+    (stroke (width 0) (type default))
+  )
   (wire (pts (xy 107.95 127) (xy 107.95 130.81))
     (stroke (width 0) (type default))
@@
     (stroke (width 0) (type default))
   )
-  (wire (pts (xy 83.82 100.33) (xy 85.09 100.33))
-    (stroke (width 0) (type default))
-  )
   (wire (pts (xy 161.29 101.6) (xy 167.64 101.6))
     (stroke (width 0) (type default))
@@
     (stroke (width 0) (type default))
   )
-  (wire (pts (xy 90.17 96.52) (xy 90.17 25.4))
-    (stroke (width 0) (type default))
-  )
   (wire (pts (xy 76.2 116.84) (xy 100.33 116.84))
     (stroke (width 0) (type default))
@@
     (stroke (width 0) (type default))
   )
-  (wire (pts (xy 43.18 100.33) (xy 83.82 100.33))
-    (stroke (width 0) (type default))
-  )
   (wire (pts (xy 167.64 71.12) (xy 167.64 74.93))
     (stroke (width 0) (type default))
@@
     (stroke (width 0) (type default))
   )
-  (wire (pts (xy 96.52 100.33) (xy 96.52 147.32))
-    (stroke (width 0) (type default))
-  )
   (wire (pts (xy 162.56 62.23) (xy 162.56 68.58))
     (stroke (width 0) (type default))
@@
   )
   (wire (pts (xy 137.16 144.78) (xy 137.16 147.32))
+    (stroke (width 0) (type default))
+  )
+  (wire (pts (xy 90.17 25.4) (xy 90.17 100.33))
     (stroke (width 0) (type default))
   )
@@
         )
       )
-    )
-  )
-  (symbol (lib_id "Jumper:Jumper_3_Bridged12") (at 90.17 100.33 180) (unit 1)
-    (in_bom yes) (on_board yes) (dnp no)
-    (property "Reference" "JP1" (at 87.63 97.79 0)
-      (effects (font (size 1.27 1.27)))
-    )
-    (property "Value" "RX Clock" (at 88.9 102.87 0)
-      (effects (font (size 1.27 1.27)))
-    )
-    (property "Footprint" "" (at 90.17 100.33 0)
-      (effects (font (size 1.27 1.27)) hide)
-    )
-    (property "Datasheet" "~" (at 90.17 100.33 0)
-      (effects (font (size 1.27 1.27)) hide)
-    )
-    (pin "1")
-    (pin "2")
-    (pin "3")
-    (instances
-      (project "ADX-ddsPIO"
-        (path "/3d934ad3-6b38-43fd-a9f4-644d18f6ed19"
-          (reference "JP1") (unit 1)
-        )
-      )

Commit message: dualclk
Connections:
- net RXIF is gone; now on net RXIF/RF(Q): TP6.1, U3.20 (GP15)
- net RFOUT: now also U3.17 (GP13); no longer U3.19 (GP14)
- net RXIF/RF(Q): now reaches C20.1, TP8.1
- net RXIF/RF(Q): now also U3.19 (GP14); no longer U3.17 (GP13)
