File: PCB/ADX-ddsPIO_V1.x.kicad_sch (KiCad schematic)
At the start: 76 parts, among them J1 Conn_Coaxial, J2 +12V, Q1 BS170, Q2 BS170, Q3 BS170, Q5 BS170, U1 L7805, U2 74LS244, U4 CD2003GB_GP, Y1 Resonator_Small

Commit message: ADX-ddsPIO_V1.3
Parts:
- removed C9: 470n, symbol Device:C
- removed D11: 1N4007, Diode_THT:D_DO-41_SOD81_P10.16mm_Horizontal, symbol Diode:1N4007
- removed Y1: Resonator_Small, symbol Device:Resonator_Small
- added C8: 470n, symbol Device:C
Connections:
- net RXA: now also C8.1
- net at C12.1, C13.1, C16.1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: now also U4.7 (AM_IF)
- net RXIF: no longer names the net of U4.4 (AM_MIX)
- net RXIF: now also C8.2
Other:
- note added: "ADX-ddsPIO digital transceiver (superhet receiver)"
- note removed: "ADX-ddsPIO digital transceiver (direct conversion receiver)"
- moved on the sheet: R17, TP4
